Commit message: fix(sd05): 消除低层速度反馈振荡
将 OCS2 默认速度阻尼从 5.5 调整为 2.0，避免 1 kHz 控制周期下速度和力矩交替发散。

增加低层力矩分项状态接口、Gazebo 接触真值和固定基座单关节测试工具，用于复现并量化振荡。

验证三个受影响包编译通过；零速度 trot 测试中前 100 ms 无强速度反向、8 秒内无力矩饱和且最大姿态偏移为 0.732 度。

File: descriptions/sd05/sd05_description/xacro/robot.xacro (robot description, xacro)
@@ -5,4 +5,12 @@
   <xacro:arg name="LOW_POLY_VISUALS" default="true"/>
   <xacro:arg name="SIMPLIFIED_VISUALS" default="false"/>
+  <xacro:arg name="FIXED_BASE" default="false"/>
+  <xacro:if value="$(arg FIXED_BASE)">
+    <link name="world"/>
+    <joint name="world_to_base" type="fixed">
+      <parent link="world"/>
+      <child link="base"/>
+    </joint>
+  </xacro:if>
   <link name="base">
     <visual>
@@ -48,4 +56,7 @@
       <xacro:include filename="$(find sd05_description)/xacro/gazebo_classic.xacro"/>
     </xacro:if>
+    <xacro:unless value="$(arg CLASSIC)">
+      <xacro:include filename="$(find sd05_description)/xacro/gazebo.xacro"/>
+    </xacro:unless>
   </xacro:if>
   <xacro:unless value="$(arg GAZEBO)">
