Commit message: feat(sd05): 添加 Gazebo 低面数显示模型
为 29 个 SD05 visual 生成 Gazebo 专用低面数 STL，原始网格保持不变，非 Gazebo 模式继续使用原始模型。

减面脚本采用二次误差度量并根据包围盒偏差自适应提高保留比例，同时生成面数、文件大小和轮廓偏差清单。总面数由 4322337 降至 799439，文件大小由约 206 MiB 降至约 38 MiB。

导出本地 Gazebo 模型搜索路径；已验证四种 Xacro 显示模式、29 个生成网格和 check_urdf。

File: descriptions/sd05/sd05_description/xacro/const.xacro (robot description, xacro)
@@ -12,5 +12,15 @@
         <origin xyz="${mesh_xyz}" rpy="0 0 0" />
         <geometry>
-          <mesh filename="${mesh}" />
+          <xacro:if value="$(arg GAZEBO)">
+            <xacro:if value="$(arg LOW_POLY_VISUALS)">
+              <mesh filename="${mesh.replace('/meshes/', '/meshes/gazebo/')}" />
+            </xacro:if>
+            <xacro:unless value="$(arg LOW_POLY_VISUALS)">
+              <mesh filename="${mesh}" />
+            </xacro:unless>
+          </xacro:if>
+          <xacro:unless value="$(arg GAZEBO)">
+            <mesh filename="${mesh}" />
+          </xacro:unless>
         </geometry>
       </xacro:unless>

File: descriptions/sd05/sd05_description/xacro/robot.xacro (robot description, xacro)
@@ -3,4 +3,5 @@
   <xacro:arg name="GAZEBO" default="false"/>
   <xacro:arg name="CLASSIC" default="false"/>
+  <xacro:arg name="LOW_POLY_VISUALS" default="true"/>
   <xacro:arg name="SIMPLIFIED_VISUALS" default="false"/>
   <link name="base">

Commit message: feat(sim): 增加SD05足端地面力诊断
为Gazebo模型增加独立接触垫和力矩传感器，在保持足端总质量与惯量不变的前提下分离地面接触力。

硬件插件发布原足端固定关节及接触垫六维力诊断话题，录包脚本同步记录相关数据；诊断接触垫不导出为控制器状态接口。

File: descriptions/sd05/sd05_description/xacro/const.xacro (robot description, xacro)
@@ -99,6 +99,12 @@
     <inertial>
       <origin xyz="0 0 0" rpy="0 0 0" />
-      <mass value="0.037" />
-      <inertia ixx="0.00000757" ixy="0" ixz="-0.00000113" iyy="0.0000076" iyz="0" izz="0.00000769" />
+      <xacro:if value="$(arg GAZEBO)">
+        <mass value="0.036" />
+        <inertia ixx="0.00000732" ixy="0" ixz="-0.00000113" iyy="0.00000735" iyz="0" izz="0.00000744" />
+      </xacro:if>
+      <xacro:unless value="$(arg GAZEBO)">
+        <mass value="0.037" />
+        <inertia ixx="0.00000757" ixy="0" ixz="-0.00000113" iyy="0.0000076" iyz="0" izz="0.00000769" />
+      </xacro:unless>
     </inertial>
     <xacro:sd05_visual mesh="package://sd05_description/meshes/FL_foot_Link.STL"
@@ -108,10 +114,12 @@
       <sphere radius="0.025" />
     </xacro:sd05_visual>
-    <collision>
-      <origin xyz="0.0 0.0 0.0" rpy="0 0 0" />
-      <geometry>
-        <sphere radius="0.025" />
-      </geometry>
-    </collision>
+    <xacro:unless value="$(arg GAZEBO)">
+      <collision>
+        <origin xyz="0.0 0.0 0.0" rpy="0 0 0" />
+        <geometry>
+          <sphere radius="0.025" />
+        </geometry>
+      </collision>
+    </xacro:unless>
   </link>
   <link name="FL_calf_rotor">
@@ -208,6 +216,12 @@
     <inertial>
       <origin xyz="0 0 0" rpy="0 0 0" />
-      <mass value="0.037" />
-      <inertia ixx="0.00000757" ixy="0" ixz="-0.00000113" iyy="0.0000076" iyz="0" izz="0.00000769" />
+      <xacro:if value="$(arg GAZEBO)">
+        <mass value="0.036" />
+        <inertia ixx="0.00000732" ixy="0" ixz="-0.00000113" iyy="0.00000735" iyz="0" izz="0.00000744" />
+      </xacro:if>
+      <xacro:unless value="$(arg GAZEBO)">
+        <mass value="0.037" />
+        <inertia ixx="0.00000757" ixy="0" ixz="-0.00000113" iyy="0.0000076" iyz="0" izz="0.00000769" />
+      </xacro:unless>
     </inertial>
     <xacro:sd05_visual mesh="package://sd05_description/meshes/FR_foot_Link.STL"
@@ -217,10 +231,12 @@
       <sphere radius="0.025" />
     </xacro:sd05_visual>
-    <collision>
-      <origin xyz="0.0 0.0 0.0" rpy="0 0 0" />
-      <geometry>
-        <sphere radius="0.025" />
-      </geometry>
-    </collision>
+    <xacro:unless value="$(arg GAZEBO)">
+      <collision>
+        <origin xyz="0.0 0.0 0.0" rpy="0 0 0" />
+        <geometry>
+          <sphere radius="0.025" />
+        </geometry>
+      </collision>
+    </xacro:unless>
   </link>
   <link name="FR_calf_rotor">
@@ -317,6 +333,12 @@
     <inertial>
       <origin xyz="0 0 0" rpy="0 0 0" />
-      <mass value="0.037" />
-      <inertia ixx="0.00000762" ixy="0" ixz="-0.00000113" iyy="0.0000076" iyz="0" izz="0.00000764" />
+      <xacro:if value="$(arg GAZEBO)">
+        <mass value="0.036" />
+        <inertia ixx="0.00000737" ixy="0" ixz="-0.00000113" iyy="0.00000735" iyz="0" izz="0.00000739" />
+      </xacro:if>
+      <xacro:unless value="$(arg GAZEBO)">
+        <mass value="0.037" />
+        <inertia ixx="0.00000762" ixy="0" ixz="-0.00000113" iyy="0.0000076" iyz="0" izz="0.00000764" />
+      </xacro:unless>
     </inertial>
     <xacro:sd05_visual mesh="package://sd05_description/meshes/RL_foot_Link.STL"
@@ -326,10 +348,12 @@
       <sphere radius="0.025" />
     </xacro:sd05_visual>
-    <collision>
-      <origin xyz="0.0 0.0 0.0" rpy="0 0 0" />
-      <geometry>
-        <sphere radius="0.025" />
-      </geometry>
-    </collision>
+    <xacro:unless value="$(arg GAZEBO)">
+      <collision>
+        <origin xyz="0.0 0.0 0.0" rpy="0 0 0" />
+        <geometry>
+          <sphere radius="0.025" />
+        </geometry>
+      </collision>
+    </xacro:unless>
   </link>
   <link name="RL_calf_rotor">
@@ -426,6 +450,12 @@
     <inertial>
       <origin xyz="0 0 0" rpy="0 0 0" />
-      <mass value="0.037" />
-      <inertia ixx="0.00000762" ixy="0" ixz="-0.00000113" iyy="0.0000076" iyz="0" izz="0.00000764" />
+      <xacro:if value="$(arg GAZEBO)">
+        <mass value="0.036" />
+        <inertia ixx="0.00000737" ixy="0" ixz="-0.00000113" iyy="0.00000735" iyz="0" izz="0.00000739" />
+      </xacro:if>
+      <xacro:unless value="$(arg GAZEBO)">
+        <mass value="0.037" />
+        <inertia ixx="0.00000762" ixy="0" ixz="-0.00000113" iyy="0.0000076" iyz="0" izz="0.00000764" />
+      </xacro:unless>
     </inertial>
     <xacro:sd05_visual mesh="package://sd05_description/meshes/RR_foot_Link.STL"
@@ -435,10 +465,12 @@
       <sphere radius="0.025" />
     </xacro:sd05_visual>
-    <collision>
-      <origin xyz="0.0 0.0 0.0" rpy="0 0 0" />
-      <geometry>
-        <sphere radius="0.025" />
-      </geometry>
-    </collision>
+    <xacro:unless value="$(arg GAZEBO)">
+      <collision>
+        <origin xyz="0.0 0.0 0.0" rpy="0 0 0" />
+        <geometry>
+          <sphere radius="0.025" />
+        </geometry>
+      </collision>
+    </xacro:unless>
   </link>
   <link name="RR_calf_rotor">

File: descriptions/sd05/sd05_description/xacro/gazebo.xacro (robot description, xacro)
@@ -2,13 +2,34 @@
 <robot xmlns:xacro="http://www.ros.org/wiki/xacro">
   <xacro:include filename="$(find gz_quadruped_hardware)/xacro/foot_force_sensor.xacro"/>
-  <xacro:macro name="foot_contact_sensor" params="name">
-    <gazebo reference="${name}_foot">
-      <sensor name="${name}_foot_contact" type="contact">
+  <xacro:macro name="foot_contact_pad" params="name">
+    <link name="${name}_contact_pad">
+      <inertial>
+        <origin xyz="0 0 0" rpy="0 0 0"/>
+        <mass value="0.001"/>
+        <inertia ixx="0.00000025" ixy="0" ixz="0"
+                 iyy="0.00000025" iyz="0" izz="0.00000025"/>
+      </inertial>
+      <collision>
+        <origin xyz="0 0 0" rpy="0 0 0"/>
+        <geometry>
+          <sphere radius="0.025"/>
+        </geometry>
+      </collision>
+    </link>
+    <joint name="${name}_contact_sensor_joint" type="fixed">
+      <origin xyz="0 0 0" rpy="0 0 0"/>
+      <parent link="${name}_foot"/>
+      <child link="${name}_contact_pad"/>
+    </joint>
+    <gazebo reference="${name}_contact_sensor_joint">
+      <provide_feedback>true</provide_feedback>
+      <disableFixedJointLumping>true</disableFixedJointLumping>
+      <sensor name="${name}_contact_pad_wrench" type="force_torque">
         <always_on>1</always_on>
         <update_rate>1000</update_rate>
-        <contact>
-          <collision>${name}_foot_collision</collision>
-          <topic>${name}_foot_contact</topic>
-        </contact>
+        <topic>${name}_contact_pad_wrench</topic>
+        <force_torque>
+          <frame>child</frame>
+        </force_torque>
       </sensor>
     </gazebo>
@@ -290,7 +311,7 @@
   <xacro:foot_force_sensor name="FR" suffix="foot_joint"/>
   <xacro:foot_force_sensor name="RR" suffix="foot_joint"/>
-  <xacro:foot_contact_sensor name="FL"/>
-  <xacro:foot_contact_sensor name="FR"/>
-  <xacro:foot_contact_sensor name="RL"/>
-  <xacro:foot_contact_sensor name="RR"/>
+  <xacro:foot_contact_pad name="FL"/>
+  <xacro:foot_contact_pad name="FR"/>
+  <xacro:foot_contact_pad name="RL"/>
+  <xacro:foot_contact_pad name="RR"/>
 </robot>
