Commit message: refactor(sd05): 适配 ROS2 ament 打包
- package.xml/CMakeLists.txt 改为 ament_cmake,包名 sd05_description
- URDF/launch 中 package:// 资源路径同步改名

File: descriptions/sd05/sd05_description/urdf/SD05-20260506.urdf (robot description, URDF)
Before this commit: robot SD05-20260506, 29 links, 28 joints
Links:
- link FL_calf_Link: geometry collision box size=0.02 0.02 0.2; visual mesh filename=package://sd05_description/meshes/FL_calf_Link.STL
- link FL_calf_rotor_Link: geometry visual mesh filename=package://sd05_description/meshes/FL_calf_rotor_Link.STL
- link FL_foot_Link: geometry collision sphere radius=0.025; visual mesh filename=package://sd05_description/meshes/FL_foot_Link.STL
- link FL_hip_Link: geometry visual mesh filename=package://sd05_description/meshes/FL_hip_Link.STL
- link FL_hip_rotor_Link: geometry visual mesh filename=package://sd05_description/meshes/FL_hip_rotor_Link.STL
- link FL_thigh_Link: geometry collision box size=0.03 0.03 0.2; visual mesh filename=package://sd05_description/meshes/FL_thigh_Link.STL
- link FL_thigh_rotor_Link: geometry visual mesh filename=package://sd05_description/meshes/FL_thigh_rotor_Link.STL
- link FR_calf_Link: geometry collision mesh filename=package://sd05_description/meshes/FR_calf_Link.STL; visual mesh filename=package://sd05_description/meshes/FR_calf_Link.STL
- link FR_calf_rotor_Link: geometry visual mesh filename=package://sd05_description/meshes/FR_calf_rotor_Link.STL
- link FR_foot_Link: geometry collision mesh filename=package://sd05_description/meshes/FR_foot_Link.STL; visual mesh filename=package://sd05_description/meshes/FR_foot_Link.STL
- link FR_hip_Link: geometry visual mesh filename=package://sd05_description/meshes/FR_hip_Link.STL
- link FR_hip_rotor_Link: geometry visual mesh filename=package://sd05_description/meshes/FR_hip_rotor_Link.STL
- link FR_thigh_Link: geometry collision mesh filename=package://sd05_description/meshes/FR_thigh_Link.STL; visual mesh filename=package://sd05_description/meshes/FR_thigh_Link.STL
- link FR_thigh_rotor_Link: geometry visual mesh filename=package://sd05_description/meshes/FR_thigh_rotor_Link.STL
- link RL_calf_Link: geometry collision mesh filename=package://sd05_description/meshes/RL_calf_Link.STL; visual mesh filename=package://sd05_description/meshes/RL_calf_Link.STL
- link RL_calf_rotor_Link: geometry visual mesh filename=package://sd05_description/meshes/RL_calf_rotor_Link.STL
- link RL_foot_Link: geometry collision mesh filename=package://sd05_description/meshes/RL_foot_Link.STL; visual mesh filename=package://sd05_description/meshes/RL_foot_Link.STL
- link RL_hip_Link: geometry visual mesh filename=package://sd05_description/meshes/RL_hip_Link.STL
- link RL_hip_rotor_Link: geometry visual mesh filename=package://sd05_description/meshes/RL_hip_rotor_Link.STL
- link RL_thigh_Link: geometry collision mesh filename=package://sd05_description/meshes/RL_thigh_Link.STL; visual mesh filename=package://sd05_description/meshes/RL_thigh_Link.STL
- link RL_thigh_rotor_Link: geometry visual mesh filename=package://sd05_description/meshes/RL_thigh_rotor_Link.STL
- link RR_calf_Link: geometry collision mesh filename=package://sd05_description/meshes/RR_calf_Link.STL; visual mesh filename=package://sd05_description/meshes/RR_calf_Link.STL
- link RR_calf_rotor_Link: geometry visual mesh filename=package://sd05_description/meshes/RR_calf_rotor_Link.STL
- link RR_foot_Link: geometry collision mesh filename=package://sd05_description/meshes/RR_foot_Link.STL; visual mesh filename=package://sd05_description/meshes/RR_foot_Link.STL
- link RR_hip_Link: geometry visual mesh filename=package://sd05_description/meshes/RR_hip_Link.STL
- link RR_hip_rotor_Link: geometry visual mesh filename=package://sd05_description/meshes/RR_hip_rotor_Link.STL
- link RR_thigh_Link: geometry collision mesh filename=package://sd05_description/meshes/RR_thigh_Link.STL; visual mesh filename=package://sd05_description/meshes/RR_thigh_Link.STL
- link RR_thigh_rotor_Link: geometry visual mesh filename=package://sd05_description/meshes/RR_thigh_rotor_Link.STL
- link base_link: geometry collision box size=0.286 0.206 0.120; visual mesh filename=package://sd05_description/meshes/base_link.STL

File: descriptions/sd05/sd05_description/urdf/SD05-20260506_collision_v1.urdf (robot description, URDF)
Before this commit: robot SD05-20260506_train_collision_v9_short_legs, 29 links, 28 joints
Links:
- link FL_calf_Link: geometry collision box size=0.030 0.030 0.165; visual mesh filename=package://sd05_description/meshes/FL_calf_Link.STL
- link FL_calf_rotor_Link: geometry visual mesh filename=package://sd05_description/meshes/FL_calf_rotor_Link.STL
- link FL_foot_Link: geometry collision sphere radius=0.025; visual mesh filename=package://sd05_description/meshes/FL_foot_Link.STL
- link FL_hip_Link: geometry visual mesh filename=package://sd05_description/meshes/FL_hip_Link.STL
- link FL_hip_rotor_Link: geometry collision cylinder length=0.07 radius=0.052; visual mesh filename=package://sd05_description/meshes/FL_hip_rotor_Link.STL
- link FL_thigh_Link: geometry collision box size=0.040 0.040 0.165; visual mesh filename=package://sd05_description/meshes/FL_thigh_Link.STL
- link FL_thigh_rotor_Link: geometry visual mesh filename=package://sd05_description/meshes/FL_thigh_rotor_Link.STL
- link FR_calf_Link: geometry collision box size=0.030 0.030 0.165; visual mesh filename=package://sd05_description/meshes/FR_calf_Link.STL
- link FR_calf_rotor_Link: geometry visual mesh filename=package://sd05_description/meshes/FR_calf_rotor_Link.STL
- link FR_foot_Link: geometry collision sphere radius=0.025; visual mesh filename=package://sd05_description/meshes/FR_foot_Link.STL
- link FR_hip_Link: geometry visual mesh filename=package://sd05_description/meshes/FR_hip_Link.STL
- link FR_hip_rotor_Link: geometry collision cylinder length=0.070 radius=0.052; visual mesh filename=package://sd05_description/meshes/FR_hip_rotor_Link.STL
- link FR_thigh_Link: geometry collision box size=0.040 0.040 0.165; visual mesh filename=package://sd05_description/meshes/FR_thigh_Link.STL
- link FR_thigh_rotor_Link: geometry visual mesh filename=package://sd05_description/meshes/FR_thigh_rotor_Link.STL
- link RL_calf_Link: geometry collision box size=0.030 0.030 0.165; visual mesh filename=package://sd05_description/meshes/RL_calf_Link.STL
- link RL_calf_rotor_Link: geometry visual mesh filename=package://sd05_description/meshes/RL_calf_rotor_Link.STL
- link RL_foot_Link: geometry collision sphere radius=0.025; visual mesh filename=package://sd05_description/meshes/RL_foot_Link.STL
- link RL_hip_Link: geometry visual mesh filename=package://sd05_description/meshes/RL_hip_Link.STL
- link RL_hip_rotor_Link: geometry collision cylinder length=0.080 radius=0.052; visual mesh filename=package://sd05_description/meshes/RL_hip_rotor_Link.STL
- link RL_thigh_Link: geometry collision box size=0.040 0.040 0.165; visual mesh filename=package://sd05_description/meshes/RL_thigh_Link.STL
- link RL_thigh_rotor_Link: geometry visual mesh filename=package://sd05_description/meshes/RL_thigh_rotor_Link.STL
- link RR_calf_Link: geometry collision box size=0.030 0.030 0.165; visual mesh filename=package://sd05_description/meshes/RR_calf_Link.STL
- link RR_calf_rotor_Link: geometry visual mesh filename=package://sd05_description/meshes/RR_calf_rotor_Link.STL
- link RR_foot_Link: geometry collision sphere radius=0.025; visual mesh filename=package://sd05_description/meshes/RR_foot_Link.STL
- link RR_hip_Link: geometry visual mesh filename=package://sd05_description/meshes/RR_hip_Link.STL
- link RR_hip_rotor_Link: geometry collision cylinder length=0.080 radius=0.052; visual mesh filename=package://sd05_description/meshes/RR_hip_rotor_Link.STL
- link RR_thigh_Link: geometry collision box size=0.040 0.040 0.165; visual mesh filename=package://sd05_description/meshes/RR_thigh_Link.STL
- link RR_thigh_rotor_Link: geometry visual mesh filename=package://sd05_description/meshes/RR_thigh_rotor_Link.STL
- link base_link: geometry collision box size=0.270 0.245 0.15; visual mesh filename=package://sd05_description/meshes/base_link.STL

Commit message: fix(sd05): 关节扭矩限制乘以减速比 8.73
SolidWorks 导出的 effort=4 为电机侧额定扭矩,关节侧应为
4 x 8.73 = 34.92 Nm(全部 12 个驱动关节)。
velocity=15 rad/s 按关节侧保留未动(若为电机侧则折算后 1.7 rad/s
无法行走,不合理),待与电机手册核对。
顺带修正导出器产生的惯量双零前缀笔误(00.0006 -> 0.0006)。

File: descriptions/sd05/sd05_description/urdf/SD05-20260506.urdf (robot description, URDF)
Before this commit: robot SD05-20260506, 29 links, 28 joints
Joints:
- joint FL_calf_joint: limit lower=-2.875 upper=-1.3 effort=4 velocity=15 -> lower=-2.875 upper=-1.3 effort=34.92 velocity=15
- joint FL_hip_joint: limit lower=-0.87 upper=0.87 effort=4 velocity=15 -> lower=-0.87 upper=0.87 effort=34.92 velocity=15
- joint FL_thigh_joint: limit lower=-1.5 upper=4.2 effort=4 velocity=15 -> lower=-1.5 upper=4.2 effort=34.92 velocity=15
- joint FR_calf_joint: limit lower=-2.875 upper=-1.3 effort=4 velocity=15 -> lower=-2.875 upper=-1.3 effort=34.92 velocity=15
- joint FR_hip_joint: limit lower=-0.87 upper=0.87 effort=4 velocity=15 -> lower=-0.87 upper=0.87 effort=34.92 velocity=15
- joint FR_thigh_joint: limit lower=-1.5 upper=4.2 effort=4 velocity=15 -> lower=-1.5 upper=4.2 effort=34.92 velocity=15
- joint RL_calf_joint: limit lower=-2.875 upper=-1.3 effort=4 velocity=15 -> lower=-2.875 upper=-1.3 effort=34.92 velocity=15
- joint RL_hip_joint: limit lower=-0.87 upper=0.87 effort=4 velocity=15 -> lower=-0.87 upper=0.87 effort=34.92 velocity=15
- joint RL_thigh_joint: limit lower=-1.5 upper=4.2 effort=4 velocity=15 -> lower=-1.5 upper=4.2 effort=34.92 velocity=15
- joint RR_calf_joint: limit lower=-2.875 upper=-1.3 effort=4 velocity=15 -> lower=-2.875 upper=-1.3 effort=34.92 velocity=15
- joint RR_hip_joint: limit lower=-0.87 upper=0.87 effort=4 velocity=15 -> lower=-0.87 upper=0.87 effort=34.92 velocity=15
- joint RR_thigh_joint: limit lower=-1.5 upper=4.2 effort=4 velocity=15 -> lower=-1.5 upper=4.2 effort=34.92 velocity=15

File: descriptions/sd05/sd05_description/urdf/SD05-20260506_collision_v1.urdf (robot description, URDF)
Before this commit: robot SD05-20260506_train_collision_v9_short_legs, 29 links, 28 joints
Joints:
- joint FL_calf_joint: limit lower=-2.875 upper=-1.3 effort=4 velocity=15 -> lower=-2.875 upper=-1.3 effort=34.92 velocity=15
- joint FL_hip_joint: limit lower=-0.87 upper=0.87 effort=4 velocity=15 -> lower=-0.87 upper=0.87 effort=34.92 velocity=15
- joint FL_thigh_joint: limit lower=-1.5 upper=4.2 effort=4 velocity=15 -> lower=-1.5 upper=4.2 effort=34.92 velocity=15
- joint FR_calf_joint: limit lower=-2.875 upper=-1.3 effort=4 velocity=15 -> lower=-2.875 upper=-1.3 effort=34.92 velocity=15
- joint FR_hip_joint: limit lower=-0.87 upper=0.87 effort=4 velocity=15 -> lower=-0.87 upper=0.87 effort=34.92 velocity=15
- joint FR_thigh_joint: limit lower=-1.5 upper=4.2 effort=4 velocity=15 -> lower=-1.5 upper=4.2 effort=34.92 velocity=15
- joint RL_calf_joint: limit lower=-2.875 upper=-1.3 effort=4 velocity=15 -> lower=-2.875 upper=-1.3 effort=34.92 velocity=15
- joint RL_hip_joint: limit lower=-0.87 upper=0.87 effort=4 velocity=15 -> lower=-0.87 upper=0.87 effort=34.92 velocity=15
- joint RL_thigh_joint: limit lower=-1.5 upper=4.2 effort=4 velocity=15 -> lower=-1.5 upper=4.2 effort=34.92 velocity=15
- joint RR_calf_joint: limit lower=-2.875 upper=-1.3 effort=4 velocity=15 -> lower=-2.875 upper=-1.3 effort=34.92 velocity=15
- joint RR_hip_joint: limit lower=-0.87 upper=0.87 effort=4 velocity=15 -> lower=-0.87 upper=0.87 effort=34.92 velocity=15
- joint RR_thigh_joint: limit lower=-1.5 upper=4.2 effort=4 velocity=15 -> lower=-1.5 upper=4.2 effort=34.92 velocity=15

Commit message: fix(sd05): 按执行器型号修正关节力矩上限
hip和thigh采用HT8108-J6峰值17 Nm，calf采用HT8108-J9堵转22 Nm，并按外部平行四边形连杆1:1传动配置。

同步更新原始URDF、碰撞URDF、Xacro、OCS2运行URDF及WBC力矩约束。

验证URDF解析和描述包编译通过；站立及零速度trot测试未发生力矩饱和。

File: descriptions/sd05/sd05_description/urdf/SD05-20260506.urdf (robot description, URDF)
Before this commit: robot SD05-20260506, 29 links, 28 joints
Joints:
- joint FL_calf_joint: limit lower=-2.875 upper=-1.3 effort=34.92 velocity=15 -> lower=-2.875 upper=-1.3 effort=22 velocity=15
- joint FL_hip_joint: limit lower=-0.87 upper=0.87 effort=34.92 velocity=15 -> lower=-0.87 upper=0.87 effort=17 velocity=15
- joint FL_thigh_joint: limit lower=-1.5 upper=4.2 effort=34.92 velocity=15 -> lower=-1.5 upper=4.2 effort=17 velocity=15
- joint FR_calf_joint: limit lower=-2.875 upper=-1.3 effort=34.92 velocity=15 -> lower=-2.875 upper=-1.3 effort=22 velocity=15
- joint FR_hip_joint: limit lower=-0.87 upper=0.87 effort=34.92 velocity=15 -> lower=-0.87 upper=0.87 effort=17 velocity=15
- joint FR_thigh_joint: limit lower=-1.5 upper=4.2 effort=34.92 velocity=15 -> lower=-1.5 upper=4.2 effort=17 velocity=15
- joint RL_calf_joint: limit lower=-2.875 upper=-1.3 effort=34.92 velocity=15 -> lower=-2.875 upper=-1.3 effort=22 velocity=15
- joint RL_hip_joint: limit lower=-0.87 upper=0.87 effort=34.92 velocity=15 -> lower=-0.87 upper=0.87 effort=17 velocity=15
- joint RL_thigh_joint: limit lower=-1.5 upper=4.2 effort=34.92 velocity=15 -> lower=-1.5 upper=4.2 effort=17 velocity=15
- joint RR_calf_joint: limit lower=-2.875 upper=-1.3 effort=34.92 velocity=15 -> lower=-2.875 upper=-1.3 effort=22 velocity=15
- joint RR_hip_joint: limit lower=-0.87 upper=0.87 effort=34.92 velocity=15 -> lower=-0.87 upper=0.87 effort=17 velocity=15
- joint RR_thigh_joint: limit lower=-1.5 upper=4.2 effort=34.92 velocity=15 -> lower=-1.5 upper=4.2 effort=17 velocity=15

File: descriptions/sd05/sd05_description/urdf/SD05-20260506_collision_v1.urdf (robot description, URDF)
Before this commit: robot SD05-20260506_train_collision_v9_short_legs, 29 links, 28 joints
Joints:
- joint FL_calf_joint: limit lower=-2.875 upper=-1.3 effort=34.92 velocity=15 -> lower=-2.875 upper=-1.3 effort=22 velocity=15
- joint FL_hip_joint: limit lower=-0.87 upper=0.87 effort=34.92 velocity=15 -> lower=-0.87 upper=0.87 effort=17 velocity=15
- joint FL_thigh_joint: limit lower=-1.5 upper=4.2 effort=34.92 velocity=15 -> lower=-1.5 upper=4.2 effort=17 velocity=15
- joint FR_calf_joint: limit lower=-2.875 upper=-1.3 effort=34.92 velocity=15 -> lower=-2.875 upper=-1.3 effort=22 velocity=15
- joint FR_hip_joint: limit lower=-0.87 upper=0.87 effort=34.92 velocity=15 -> lower=-0.87 upper=0.87 effort=17 velocity=15
- joint FR_thigh_joint: limit lower=-1.5 upper=4.2 effort=34.92 velocity=15 -> lower=-1.5 upper=4.2 effort=17 velocity=15
- joint RL_calf_joint: limit lower=-2.875 upper=-1.3 effort=34.92 velocity=15 -> lower=-2.875 upper=-1.3 effort=22 velocity=15
- joint RL_hip_joint: limit lower=-0.87 upper=0.87 effort=34.92 velocity=15 -> lower=-0.87 upper=0.87 effort=17 velocity=15
- joint RL_thigh_joint: limit lower=-1.5 upper=4.2 effort=34.92 velocity=15 -> lower=-1.5 upper=4.2 effort=17 velocity=15
- joint RR_calf_joint: limit lower=-2.875 upper=-1.3 effort=34.92 velocity=15 -> lower=-2.875 upper=-1.3 effort=22 velocity=15
- joint RR_hip_joint: limit lower=-0.87 upper=0.87 effort=34.92 velocity=15 -> lower=-0.87 upper=0.87 effort=17 velocity=15
- joint RR_thigh_joint: limit lower=-1.5 upper=4.2 effort=34.92 velocity=15 -> lower=-1.5 upper=4.2 effort=17 velocity=15

File: descriptions/sd05/sd05_description/urdf/robot.urdf (robot description, URDF)
Before this commit: robot sd05, 31 links, 30 joints
Joints:
- joint FL_calf_joint: limit lower=-2.875 upper=-1.3 effort=34.92 velocity=15 -> lower=-2.875 upper=-1.3 effort=22 velocity=15
- joint FL_hip_joint: limit lower=-0.87 upper=0.87 effort=34.92 velocity=15 -> lower=-0.87 upper=0.87 effort=17 velocity=15
- joint FL_thigh_joint: limit lower=-1.5 upper=4.2 effort=34.92 velocity=15 -> lower=-1.5 upper=4.2 effort=17 velocity=15
- joint FR_calf_joint: limit lower=-2.875 upper=-1.3 effort=34.92 velocity=15 -> lower=-2.875 upper=-1.3 effort=22 velocity=15
- joint FR_hip_joint: limit lower=-0.87 upper=0.87 effort=34.92 velocity=15 -> lower=-0.87 upper=0.87 effort=17 velocity=15
- joint FR_thigh_joint: limit lower=-1.5 upper=4.2 effort=34.92 velocity=15 -> lower=-1.5 upper=4.2 effort=17 velocity=15
- joint RL_calf_joint: limit lower=-2.875 upper=-1.3 effort=34.92 velocity=15 -> lower=-2.875 upper=-1.3 effort=22 velocity=15
- joint RL_hip_joint: limit lower=-0.87 upper=0.87 effort=34.92 velocity=15 -> lower=-0.87 upper=0.87 effort=17 velocity=15
- joint RL_thigh_joint: limit lower=-1.5 upper=4.2 effort=34.92 velocity=15 -> lower=-1.5 upper=4.2 effort=17 velocity=15
- joint RR_calf_joint: limit lower=-2.875 upper=-1.3 effort=34.92 velocity=15 -> lower=-2.875 upper=-1.3 effort=22 velocity=15
- joint RR_hip_joint: limit lower=-0.87 upper=0.87 effort=34.92 velocity=15 -> lower=-0.87 upper=0.87 effort=17 velocity=15
- joint RR_thigh_joint: limit lower=-1.5 upper=4.2 effort=34.92 velocity=15 -> lower=-1.5 upper=4.2 effort=17 velocity=15

File: descriptions/sd05/sd05_description/xacro/const.xacro (robot description, xacro)
@@ -489,5 +489,5 @@
     <child link="FL_hip" />
     <axis xyz="1 0 0" />
-    <limit lower="-0.87" upper="0.87" effort="34.92" velocity="15" />
+    <limit lower="-0.87" upper="0.87" effort="17" velocity="15" />
   </joint>
   <joint name="FL_thigh_joint" type="revolute">
@@ -496,5 +496,5 @@
     <child link="FL_thigh" />
     <axis xyz="0 1 0" />
-    <limit lower="-1.5" upper="4.2" effort="34.92" velocity="15" />
+    <limit lower="-1.5" upper="4.2" effort="17" velocity="15" />
   </joint>
   <joint name="FL_calf_joint" type="revolute">
@@ -503,5 +503,5 @@
     <child link="FL_calf" />
     <axis xyz="0 1 0" />
-    <limit lower="-2.875" upper="-1.3" effort="34.92" velocity="15" />
+    <limit lower="-2.875" upper="-1.3" effort="22" velocity="15" />
   </joint>
   <joint name="FL_foot_joint" type="fixed">
@@ -534,5 +534,5 @@
     <child link="FR_hip" />
     <axis xyz="1 0 0" />
-    <limit lower="-0.87" upper="0.87" effort="34.92" velocity="15" />
+    <limit lower="-0.87" upper="0.87" effort="17" velocity="15" />
   </joint>
   <joint name="FR_thigh_joint" type="revolute">
@@ -541,5 +541,5 @@
     <child link="FR_thigh" />
     <axis xyz="0 1 0" />
-    <limit lower="-1.5" upper="4.2" effort="34.92" velocity="15" />
+    <limit lower="-1.5" upper="4.2" effort="17" velocity="15" />
   </joint>
   <joint name="FR_calf_joint" type="revolute">
@@ -548,5 +548,5 @@
     <child link="FR_calf" />
     <axis xyz="0 1 0" />
-    <limit lower="-2.875" upper="-1.3" effort="34.92" velocity="15" />
+    <limit lower="-2.875" upper="-1.3" effort="22" velocity="15" />
   </joint>
   <joint name="FR_foot_joint" type="fixed">
@@ -579,5 +579,5 @@
     <child link="RL_hip" />
     <axis xyz="1 0 0" />
-    <limit lower="-0.87" upper="0.87" effort="34.92" velocity="15" />
+    <limit lower="-0.87" upper="0.87" effort="17" velocity="15" />
   </joint>
   <joint name="RL_thigh_joint" type="revolute">
@@ -586,5 +586,5 @@
     <child link="RL_thigh" />
     <axis xyz="0 1 0" />
-    <limit lower="-1.5" upper="4.2" effort="34.92" velocity="15" />
+    <limit lower="-1.5" upper="4.2" effort="17" velocity="15" />
   </joint>
   <joint name="RL_calf_joint" type="revolute">
@@ -593,5 +593,5 @@
     <child link="RL_calf" />
     <axis xyz="0 1 0" />
-    <limit lower="-2.875" upper="-1.3" effort="34.92" velocity="15" />
+    <limit lower="-2.875" upper="-1.3" effort="22" velocity="15" />
   </joint>
   <joint name="RL_foot_joint" type="fixed">
@@ -624,5 +624,5 @@
     <child link="RR_hip" />
     <axis xyz="1 0 0" />
-    <limit lower="-0.87" upper="0.87" effort="34.92" velocity="15" />
+    <limit lower="-0.87" upper="0.87" effort="17" velocity="15" />
   </joint>
   <joint name="RR_thigh_joint" type="revolute">
@@ -631,5 +631,5 @@
     <child link="RR_thigh" />
     <axis xyz="0 1 0" />
-    <limit lower="-1.5" upper="4.2" effort="34.92" velocity="15" />
+    <limit lower="-1.5" upper="4.2" effort="17" velocity="15" />
   </joint>
   <joint name="RR_calf_joint" type="revolute">
@@ -638,5 +638,5 @@
     <child link="RR_calf" />
     <axis xyz="0 1 0" />
-    <limit lower="-2.875" upper="-1.3" effort="34.92" velocity="15" />
+    <limit lower="-2.875" upper="-1.3" effort="22" velocity="15" />
   </joint>
   <joint name="RR_foot_joint" type="fixed">
